Commit message: URDFからガゼボ関連のプラグイン排除した。

File: urdf/sirius3.urdf copy.xacro (robot description, xacro)
@@ -156,3 +156,102 @@
     <child link="$(arg prefix)lidar_link" />
   </joint>
+  <!-- Gazebo関連の設定 -->
+  <gazebo reference="$(arg prefix)base_link">
+    <material>Gazebo/Blue</material>
+    <mu1>0.5</mu1>
+    <mu2>0.8</mu2>
+  </gazebo>
+  <gazebo reference="$(arg prefix)left_wheel">
+    <material>Gazebo/Grey</material>
+    <mu1>1.5</mu1>
+    <mu2>1.5</mu2>
+  </gazebo>
+  <gazebo reference="$(arg prefix)right_wheel">
+    <material>Gazebo/Grey</material>
+    <mu1>1.5</mu1>
+    <mu2>1.5</mu2>
+  </gazebo>
+  <gazebo reference="$(arg prefix)lidar_link">
+    <material>Gazebo/Grey</material>
+  </gazebo>
+  <!-- Gazebo Plugins -->
+  <!-- Differential Drive Plugin -->
+  <gazebo>
+    <plugin name="differential_drive_controller" filename="libgazebo_ros_diff_drive.so">
+      <ros>
+        <namespace>/sirius3</namespace>
+        <argument>--ros-args --remap cmd_vel:=cmd_vel</argument>
+        <argument>--ros-args --remap odom:=odom</argument>
+      </ros>
+      <!-- ジョイント名 -->
+      <left_joint>$(arg prefix)left_wheel_joint</left_joint>
+      <right_joint>$(arg prefix)right_wheel_joint</right_joint>
+      <!-- 車輪パラメータ -->
+      <wheel_separation>${wheel_separation}</wheel_separation>
+      <wheel_diameter>${wheel_radius * 2}</wheel_diameter>
+      <!-- コマンド入力トピック -->
+      <command_topic>cmd_vel</command_topic>
+      <!-- オドメトリ -->
+      <publish_odom>true</publish_odom>
+      <publish_odom_tf>true</publish_odom_tf>
+      <publish_wheel_tf>false</publish_wheel_tf>
+      <odometry_frame>odom</odometry_frame>
+      <robot_base_frame>$(arg prefix)base_footprint</robot_base_frame>
+      <!-- 更新頻度 -->
+      <update_rate>50</update_rate>
+      <!-- 最大速度 -->
+      <max_wheel_torque>100</max_wheel_torque>
+      <max_wheel_acceleration>1.0</max_wheel_acceleration>
+      <!-- オドメトリノイズ -->
+      <odometry_source>world</odometry_source>
+    </plugin>
+  </gazebo>
+  <!-- LiDAR Sensor Plugin -->
+  <gazebo reference="$(arg prefix)lidar_link">
+    <sensor type="gpu_ray" name="lidar_sensor">
+      <pose>0 0 0 0 0 0</pose>
+      <visualize>true</visualize>
+      <update_rate>10</update_rate>
+      <ray>
+        <scan>
+          <horizontal>
+            <samples>360</samples>
+            <resolution>1</resolution>
+            <min_angle>-3.14159</min_angle>
+            <max_angle>3.14159</max_angle>
+          </horizontal>
+        </scan>
+        <range>
+          <min>0.1</min>
+          <max>100.0</max>
+          <resolution>0.01</resolution>
+        </range>
+        <noise>
+          <type>gaussian</type>
+          <mean>0.0</mean>
+          <stddev>0.01</stddev>
+        </noise>
+      </ray>
+      <plugin name="gazebo_ros_lidar_controller" filename="libgazebo_ros_ray_sensor.so">
+        <ros>
+          <namespace>/sirius3</namespace>
+          <argument>--ros-args --remap ~/out:=scan</argument>
+        </ros>
+        <output_type>sensor_msgs/LaserScan</output_type>
+        <frame_name>$(arg prefix)lidar_link</frame_name>
+      </plugin>
+    </sensor>
+  </gazebo>
+  <!-- Joint State Publisher -->
+  <gazebo>
+    <plugin name="gazebo_ros_joint_state_publisher" filename="libgazebo_ros_joint_state_publisher.so">
+      <ros>
+        <namespace>/sirius3</namespace>
+        <argument>--ros-args --remap joint_states:=joint_states</argument>
+      </ros>
+      <update_rate>50</update_rate>
+      <joint_name>$(arg prefix)left_wheel_joint</joint_name>
+      <joint_name>$(arg prefix)right_wheel_joint</joint_name>
+    </plugin>
+  </gazebo>
 </robot>
