Commit message: これでとりあえずおけ。ただし、 sirius3/left_wheel No transform from [sirius3/left_wheel] to [sirius3/odom]

File: urdf/sirius3.urdf.xacro (robot description, xacro)
@@ -76,5 +76,5 @@
       </collision>
     </link>
-    <joint name="$(arg prefix)${side}_wheel_joint" type="continuous">
+    <joint name="${side}_wheel_joint" type="continuous">
       <origin xyz="${joint_origin}" rpy="${joint_rpy}" />
       <parent link="$(arg prefix)base_link" />

Commit message: とりあえず、できた。次はLiDARつける。

File: urdf/sirius3.urdf.xacro (robot description, xacro)
@@ -51,5 +51,5 @@
     <parent link="$(arg prefix)base_footprint"/>
     <child link="$(arg prefix)base_link"/>
-    <origin xyz="0 0 0" rpy="0 0 0"/>
+    <origin xyz="0 0 0" rpy="0 0 1.5707963267948966"/>
   </joint>
   <!-- ホイールマクロ定義 -->

Commit message: 

File: urdf/sirius3.urdf.xacro (robot description, xacro)
@@ -18,6 +18,6 @@
     <color rgba="0.1 0.3 0.6 1.0"/>
   </material>
-  <material name="wheel_gray">
-    <color rgba="0.3 0.3 0.3 1.0"/>
+  <material name="lidar_gray">
+    <color rgba="0.2 0.2 0.2 1.0"/>
   </material>
   <!-- ベースフットプリント（地面接触点の仮想リンク） -->
@@ -111,3 +111,31 @@
     axis_xyz="0.0 0.0 -1.0"
   />
+  <!-- LiDAR Link -->
+  <link name="$(arg prefix)base_link/lidar_link">
+    <inertial>
+      <origin xyz="0.0 0.0 0.0" rpy="0.0 0.0 0.0" />
+      <mass value="0.5" />
+      <inertia ixx="0.01" iyy="0.01" izz="0.01"
+               ixy="0.0" iyz="0.0" ixz="0.0" />
+    </inertial>
+    <visual name="lidar_visual">
+      <origin xyz="0.0 0.0 0.0" rpy="0.0 0.0 0.0" />
+      <geometry>
+        <cylinder radius="0.052" length="0.072" />
+      </geometry>
+      <material name="lidar_gray" />
+    </visual>
+    <collision name="lidar_collision">
+      <origin xyz="0.0 0.0 0.0" rpy="0.0 0.0 0.0" />
+      <geometry>
+        <cylinder radius="0.052" length="0.072" />
+      </geometry>
+    </collision>
+  </link>
+  <!-- LiDAR Joint -->
+  <joint name="$(arg prefix)base_link/lidar_joint" type="fixed">
+    <origin xyz="0.0 0.0 0.85" rpy="0.0 0.0 0.0" />
+    <parent link="$(arg prefix)base_link" />
+    <child link="$(arg prefix)base_link/lidar_link" />
+  </joint>
 </robot>

Commit message: meshの、車輪と回転軸を正しくしようとした。が、スケールがでかい。＋SDFではまた、手動の回転変換が必要

File: urdf/sirius3.urdf.xacro (robot description, xacro)
@@ -18,4 +18,7 @@
     <color rgba="0.1 0.3 0.6 1.0"/>
   </material>
+  <material name="wheel_gray">
+    <color rgba="0.5 0.5 0.5 1.0"/>
+  </material>
   <material name="lidar_gray">
     <color rgba="0.2 0.2 0.2 1.0"/>
@@ -36,5 +39,5 @@
       <origin xyz="0.0 0.0 0.0" rpy="0.0 0.0 0.0" />
       <geometry>
-        <mesh filename="${mesh_path}/Sirius3-body-v2.stl" scale="0.001 0.001 0.001" />
+        <mesh filename="${mesh_path}/Sirius3_body.stl" scale="0.0001 0.0001 0.0001" />
       </geometry>
       <material name="base_blue" />
@@ -43,5 +46,5 @@
       <origin xyz="0.0 0.0 0.0" rpy="0.0 0.0 0.0" />
       <geometry>
-        <mesh filename="${mesh_path}/Sirius3-body-v2.stl" scale="0.001 0.001 0.001" />
+        <mesh filename="${mesh_path}/Sirius3_body.stl" scale="0.0001 0.0001 0.0001" />
       </geometry>
     </collision>
@@ -51,5 +54,5 @@
     <parent link="$(arg prefix)base_footprint"/>
     <child link="$(arg prefix)base_link"/>
-    <origin xyz="0 0 0" rpy="0 0 1.5707963267948966"/>
+    <origin xyz="0 0 0" rpy="0 0 0"/>
   </joint>
   <!-- ホイールマクロ定義 -->
@@ -65,5 +68,5 @@
         <origin xyz="${wheel_visual_origin}" rpy="${wheel_visual_rpy}" />
         <geometry>
-          <mesh filename="${mesh_path}/${mesh_file}" scale="0.001 0.001 0.001" />
+          <mesh filename="${mesh_path}/${mesh_file}" scale="0.0001 0.0001 0.0001" />
         </geometry>
         <material name="wheel_gray" />
@@ -72,5 +75,5 @@
         <origin xyz="${wheel_visual_origin}" rpy="${wheel_visual_rpy}" />
         <geometry>
-          <mesh filename="${mesh_path}/${mesh_file}" scale="0.001 0.001 0.001" />
+          <mesh filename="${mesh_path}/${mesh_file}" scale="0.0001 0.0001 0.0001" />
         </geometry>
       </collision>
@@ -85,4 +88,17 @@
     </joint>
   </xacro:macro>
+  <!-- 右ホイール -->
+  <xacro:wheel
+    prefix="$(arg prefix)"
+    side="right"
+    reflect="-1"
+    mesh_file="Right_Wheel.stl"
+    wheel_origin_rpy="0.0 0.0 0.0"
+    wheel_visual_origin="0.0 0.0 0.0"
+    wheel_visual_rpy="0.0 0.0 1.5707963267948966"
+    joint_origin="-1.809999996270403 -0.015078560389649666 1.3253258500000007"
+    joint_rpy="-1.5707963267948997 -1.5707963267948963 0"
+    axis_xyz="0.0 -1.0 3.944304526105057e-31"
+  />
   <!-- 左ホイール -->
   <xacro:wheel
@@ -90,24 +106,11 @@
     side="left"
     reflect="1"
-    mesh_file="Left-Wheel-v1.stl"
+    mesh_file="Left_Wheel.stl"
     wheel_origin_rpy="0.0 0.0 0.0"
-    wheel_visual_origin="0.00026615125671387575 -0.0003525431147384645 -0.019999996185302748"
-    wheel_visual_rpy="-3.141592653589793 -1.5707963267948966 0"
-    joint_origin="0.18100000000000002 -0.0014818300000000002 0.13236434"
-    joint_rpy="-3.141592653589793 -1.5707963267948966 0"
-    axis_xyz="0.0 0.0 1.0"
-  />
-  <!-- 右ホイール -->
-  <xacro:wheel
-    prefix="$(arg prefix)"
-    side="right"
-    reflect="-1"
-    mesh_file="Right-Wheel-v1.stl"
-    wheel_origin_rpy="0.0 0.0 0.0"
-    wheel_visual_origin="-0.00011675030934453545 0.00014720826142882893 -0.019999996185302748"
-    wheel_visual_rpy="-0.3490658503988659 1.5707963267948966 0"
-    joint_origin="-0.18100000000000002 -0.0014818300000000002 0.1325"
-    joint_rpy="-0.0 -1.5707963267948966 0"
-    axis_xyz="0.0 0.0 -1.0"
+    wheel_visual_origin="0.0 0.0 0.0"
+    wheel_visual_rpy="0.0 0.0 3.141592653589793"
+    joint_origin="1.8100000037295931 -0.015078560389660538 1.3268722499999996"
+    joint_rpy="1.5707963267948937 -1.5707963267948963 0"
+    axis_xyz="0.0 -1.0 3.944304526105057e-31"
   />
   <!-- LiDAR Link -->

Commit message: Z軸を治そうとした。が、MeshLabじゃだめ。基準からの回転じゃなくなる

File: urdf/sirius3.urdf.xacro (robot description, xacro)
@@ -19,5 +19,5 @@
   </material>
   <material name="wheel_gray">
-    <color rgba="0.5 0.5 0.5 1.0"/>
+    <color rgba="0.3 0.3 0.3 1.0"/>
   </material>
   <material name="lidar_gray">
@@ -31,13 +31,13 @@
   <link name="$(arg prefix)base_link">
     <inertial>
-      <origin xyz="0.0002947164165949175 0.09943035225547465 0.3230235286090795" rpy="0.0 0.0 0.0" />
+      <origin xyz="0.0002947164165949161 0.09943035225547472 0.3230235286090794" rpy="0.0 0.0 0.0" />
       <mass value="${base_mass}" />
-      <inertia ixx="2.8808637737854452" iyy="2.459771630191444" izz="2.1448545974410616"
-               ixy="0.000982314201767401" iyz="0.26295068207750116" ixz="-0.0034301184728964904" />
+      <inertia ixx="2.8808637737854497" iyy="2.45977163019146" izz="2.1448545974410616"
+               ixy="0.0009823142017673183" iyz="0.26295068207749944" ixz="-0.003430118472896634" />
     </inertial>
     <visual name="base_link_visual">
       <origin xyz="0.0 0.0 0.0" rpy="0.0 0.0 0.0" />
       <geometry>
-        <mesh filename="${mesh_path}/Sirius3_body.stl" scale="0.0001 0.0001 0.0001" />
+        <mesh filename="${mesh_path}/Sirius3-body-v2.stl" scale="0.001 0.001 0.001" />
       </geometry>
       <material name="base_blue" />
@@ -46,5 +46,5 @@
       <origin xyz="0.0 0.0 0.0" rpy="0.0 0.0 0.0" />
       <geometry>
-        <mesh filename="${mesh_path}/Sirius3_body.stl" scale="0.0001 0.0001 0.0001" />
+        <mesh filename="${mesh_path}/Sirius3-body-v2.stl" scale="0.001 0.001 0.001" />
       </geometry>
     </collision>
@@ -57,16 +57,16 @@
   </joint>
   <!-- ホイールマクロ定義 -->
-  <xacro:macro name="wheel" params="prefix side reflect mesh_file wheel_origin_rpy wheel_visual_origin wheel_visual_rpy joint_origin joint_rpy axis_xyz">
+  <xacro:macro name="wheel" params="prefix side reflect mesh_file wheel_mass_value wheel_inertia_ixx wheel_inertia_iyy wheel_inertia_izz wheel_inertia_ixy wheel_inertia_iyz wheel_inertia_ixz wheel_inertial_origin wheel_visual_origin wheel_visual_rpy joint_origin joint_rpy axis_xyz">
     <link name="$(arg prefix)${side}_wheel">
       <inertial>
-        <origin xyz="0.0 0.0 0.021535" rpy="0.0 0.0 0.0" />
-        <mass value="${wheel_mass}" />
-        <inertia ixx="0.13042" iyy="0.13041" izz="0.24145"
-                 ixy="0.0" iyz="0.0" ixz="0.0" />
+        <origin xyz="${wheel_inertial_origin}" rpy="0.0 0.0 0.0" />
+        <mass value="${wheel_mass_value}" />
+        <inertia ixx="${wheel_inertia_ixx}" iyy="${wheel_inertia_iyy}" izz="${wheel_inertia_izz}"
+                 ixy="${wheel_inertia_ixy}" iyz="${wheel_inertia_iyz}" ixz="${wheel_inertia_ixz}" />
       </inertial>
       <visual name="${side}_wheel_visual">
         <origin xyz="${wheel_visual_origin}" rpy="${wheel_visual_rpy}" />
         <geometry>
-          <mesh filename="${mesh_path}/${mesh_file}" scale="0.0001 0.0001 0.0001" />
+          <mesh filename="${mesh_path}/${mesh_file}" scale="0.001 0.001 0.001" />
         </geometry>
         <material name="wheel_gray" />
@@ -75,5 +75,5 @@
         <origin xyz="${wheel_visual_origin}" rpy="${wheel_visual_rpy}" />
         <geometry>
-          <mesh filename="${mesh_path}/${mesh_file}" scale="0.0001 0.0001 0.0001" />
+          <mesh filename="${mesh_path}/${mesh_file}" scale="0.001 0.001 0.001" />
         </geometry>
       </collision>
@@ -85,7 +85,27 @@
       <axis xyz="${axis_xyz}" />
       <limit effort="100" velocity="100" />
-      <dynamics damping="0.1" friction="0.1" />
+      <dynamics damping="5.0" friction="2.0" />
     </joint>
   </xacro:macro>
+  <!-- 左ホイール -->
+  <xacro:wheel
+    prefix="$(arg prefix)"
+    side="left"
+    reflect="1"
+    mesh_file="Left-Wheel-v1.stl"
+    wheel_mass_value="26.684250609189966"
+    wheel_inertia_ixx="0.24147472596060576"
+    wheel_inertia_iyy="0.13040791997952456"
+    wheel_inertia_izz="0.13041983338763752"
+    wheel_inertia_ixy="-1.3386522533795057e-05"
+    wheel_inertia_iyz="1.9456112928556427e-05"
+    wheel_inertia_ixz="-5.293518847815378e-06"
+    wheel_inertial_origin="0.00025571114010551453 -0.02153522228931916 -0.0003576198248327911"
+    wheel_visual_origin="0.00026615125671401783 0.019999997439497593 -0.0003525390265766926"
+    wheel_visual_rpy="-1.5707963267948966 -1.5265566588595898e-16 -1.5707963267948966"
+    joint_origin="0.18100000125419488 -0.0014818259118381794 0.13236433999999986"
+    joint_rpy="1.5707963267948968 -1.5707963267948966 0"
+    axis_xyz="0.0 -1.0 0.0"
+  />
   <!-- 右ホイール -->
   <xacro:wheel
@@ -93,27 +113,21 @@
     side="right"
     reflect="-1"
-    mesh_file="Right_Wheel.stl"
-    wheel_origin_rpy="0.0 0.0 0.0"
-    wheel_visual_origin="0.0 0.0 0.0"
-    wheel_visual_rpy="0.0 0.0 1.5707963267948966"
-    joint_origin="-1.809999996270403 -0.015078560389649666 1.3253258500000007"
-    joint_rpy="-1.5707963267948997 -1.5707963267948963 0"
-    axis_xyz="0.0 -1.0 3.944304526105057e-31"
-  />
-  <!-- 左ホイール -->
-  <xacro:wheel
-    prefix="$(arg prefix)"
-    side="left"
-    reflect="1"
-    mesh_file="Left_Wheel.stl"
-    wheel_origin_rpy="0.0 0.0 0.0"
-    wheel_visual_origin="0.0 0.0 0.0"
-    wheel_visual_rpy="0.0 0.0 3.141592653589793"
-    joint_origin="1.8100000037295931 -0.015078560389660538 1.3268722499999996"
-    joint_rpy="1.5707963267948937 -1.5707963267948963 0"
-    axis_xyz="0.0 -1.0 3.944304526105057e-31"
+    mesh_file="Right-Wheel-v1.stl"
+    wheel_mass_value="26.680591288269447"
+    wheel_inertia_ixx="0.24143130580426037"
+    wheel_inertia_iyy="0.13037284939060423"
+    wheel_inertia_izz="0.13040416227048746"
+    wheel_inertia_ixy="-6.089214838569495e-06"
+    wheel_inertia_iyz="-2.3850804537560444e-05"
+    wheel_inertia_ixz="1.2550615379814878e-05"
+    wheel_inertial_origin="-0.00012199495468973254 -0.021535446042454894 0.0001603382139831866"
+    wheel_visual_origin="-0.00011675030934441111 0.020000004931107825 0.00014720417326699709"
+    wheel_visual_rpy="1.2217304763960306 1.5265566588595898e-16 1.5707963267948966"
+    joint_origin="-0.18100000874580505 -0.001481825911838235 0.13249999999999987"
+    joint_rpy="-1.5707963267948966 -1.5707963267948966 0"
+    axis_xyz="0.0 -1.0 0.0"
   />
   <!-- LiDAR Link -->
-  <link name="$(arg prefix)base_link/lidar_link">
+  <link name="$(arg prefix)lidar_link">
     <inertial>
       <origin xyz="0.0 0.0 0.0" rpy="0.0 0.0 0.0" />
@@ -137,8 +151,107 @@
   </link>
   <!-- LiDAR Joint -->
-  <joint name="$(arg prefix)base_link/lidar_joint" type="fixed">
+  <joint name="$(arg prefix)lidar_joint" type="fixed">
     <origin xyz="0.0 0.0 0.85" rpy="0.0 0.0 0.0" />
     <parent link="$(arg prefix)base_link" />
-    <child link="$(arg prefix)base_link/lidar_link" />
+    <child link="$(arg prefix)lidar_link" />
   </joint>
+  <!-- Gazebo関連の設定 -->
+  <gazebo reference="$(arg prefix)base_link">
+    <material>Gazebo/Blue</material>
+    <mu1>0.5</mu1>
+    <mu2>0.8</mu2>
+  </gazebo>
+  <gazebo reference="$(arg prefix)left_wheel">
+    <material>Gazebo/Grey</material>
+    <mu1>1.5</mu1>
+    <mu2>1.5</mu2>
+  </gazebo>
+  <gazebo reference="$(arg prefix)right_wheel">
+    <material>Gazebo/Grey</material>
+    <mu1>1.5</mu1>
+    <mu2>1.5</mu2>
+  </gazebo>
+  <gazebo reference="$(arg prefix)lidar_link">
+    <material>Gazebo/Grey</material>
+  </gazebo>
+  <!-- Gazebo Plugins -->
+  <!-- Differential Drive Plugin -->
+  <gazebo>
+    <plugin name="differential_drive_controller" filename="libgazebo_ros_diff_drive.so">
+      <ros>
+        <namespace>/sirius3</namespace>
+        <argument>--ros-args --remap cmd_vel:=cmd_vel</argument>
+        <argument>--ros-args --remap odom:=odom</argument>
+      </ros>
+      <!-- ジョイント名 -->
+      <left_joint>$(arg prefix)left_wheel_joint</left_joint>
+      <right_joint>$(arg prefix)right_wheel_joint</right_joint>
+      <!-- 車輪パラメータ -->
+      <wheel_separation>${wheel_separation}</wheel_separation>
+      <wheel_diameter>${wheel_radius * 2}</wheel_diameter>
+      <!-- コマンド入力トピック -->
+      <command_topic>cmd_vel</command_topic>
+      <!-- オドメトリ -->
+      <publish_odom>true</publish_odom>
+      <publish_odom_tf>true</publish_odom_tf>
+      <publish_wheel_tf>false</publish_wheel_tf>
+      <odometry_frame>odom</odometry_frame>
+      <robot_base_frame>$(arg prefix)base_footprint</robot_base_frame>
+      <!-- 更新頻度 -->
+      <update_rate>50</update_rate>
+      <!-- 最大速度 -->
+      <max_wheel_torque>100</max_wheel_torque>
+      <max_wheel_acceleration>1.0</max_wheel_acceleration>
+      <!-- オドメトリノイズ -->
+      <odometry_source>world</odometry_source>
+    </plugin>
+  </gazebo>
+  <!-- LiDAR Sensor Plugin -->
+  <gazebo reference="$(arg prefix)lidar_link">
+    <sensor type="gpu_ray" name="lidar_sensor">
+      <pose>0 0 0 0 0 0</pose>
+      <visualize>true</visualize>
+      <update_rate>10</update_rate>
+      <ray>
+        <scan>
+          <horizontal>
+            <samples>360</samples>
+            <resolution>1</resolution>
+            <min_angle>-3.14159</min_angle>
+            <max_angle>3.14159</max_angle>
+          </horizontal>
+        </scan>
+        <range>
+          <min>0.1</min>
+          <max>100.0</max>
+          <resolution>0.01</resolution>
+        </range>
+        <noise>
+          <type>gaussian</type>
+          <mean>0.0</mean>
+          <stddev>0.01</stddev>
+        </noise>
+      </ray>
+      <plugin name="gazebo_ros_lidar_controller" filename="libgazebo_ros_ray_sensor.so">
+        <ros>
+          <namespace>/sirius3</namespace>
+          <argument>--ros-args --remap ~/out:=scan</argument>
+        </ros>
+        <output_type>sensor_msgs/LaserScan</output_type>
+        <frame_name>$(arg prefix)lidar_link</frame_name>
+      </plugin>
+    </sensor>
+  </gazebo>
+  <!-- Joint State Publisher -->
+  <gazebo>
+    <plugin name="gazebo_ros_joint_state_publisher" filename="libgazebo_ros_joint_state_publisher.so">
+      <ros>
+        <namespace>/sirius3</namespace>
+        <argument>--ros-args --remap joint_states:=joint_states</argument>
+      </ros>
+      <update_rate>50</update_rate>
+      <joint_name>$(arg prefix)left_wheel_joint</joint_name>
+      <joint_name>$(arg prefix)right_wheel_joint</joint_name>
+    </plugin>
+  </gazebo>
 </robot>

Commit message: まだLiDARのリンク名が気持ち悪いがこれでよし

File: urdf/sirius3.urdf.xacro (robot description, xacro)
@@ -129,5 +129,5 @@
   />
   <!-- LiDAR Link -->
-  <link name="$(arg prefix)lidar_link">
+  <link name="$(arg prefix)base_link/lidar_link">
     <inertial>
       <origin xyz="0.0 0.0 0.0" rpy="0.0 0.0 0.0" />
@@ -154,5 +154,6 @@
     <origin xyz="0.0 0.0 0.85" rpy="0.0 0.0 0.0" />
     <parent link="$(arg prefix)base_link" />
-    <child link="$(arg prefix)lidar_link" />
+    <!-- 苦肉の策。これでGazebo上のTFと名前が重なるので無駄に増えなくなる -->
+    <child link="$(arg prefix)base_link/lidar_link" />
   </joint>
 </robot>
